File: ampli.sch (KiCad schematic (older format))
At the start: 52 parts, among them J2 Conn_01x02, J3 Conn_01x03, Q1 2N2907, Q10 TIP32, Q11 BD138, Q12 TIP31, Q13 2N2222, Q2 2N2907, Q3 2N2907, Q4 2N2222, Q5 2N2222, Q6 2N2907, Q7 2N2907, Q8 BD139, Q9 BD139, U1 Jack_Mono, U2 Relay_1CT

Commit message: version 1.7
Parts:
- removed U2: Relay_1CT, OJ-SS-112LMH2_005:OJ-SS-112HM.000_1, symbol Relay:Relay_1CT
- added U2: Relay_1CT, OJ-SS-112LMH2_005:OJ-SS-112HM.000_1, symbol relay_1ct:Relay_1CT
Changed lines of the file:
@@
 	7600 1650 7600 1800
-$Comp
-L Relay:Relay_1CT U2
-U 1 1 604E9772
-P 9400 2400
-F 0 "U2" H 9350 2467 50  0000 C CNN
-F 1 "Relay_1CT" H 9350 2376 50  0000 C CNN
-F 2 "OJ-SS-112LMH2_005:OJ-SS-112HM.000_1" H 9400 2400 50  0001 C CNN
-F 3 "" H 9400 2400 50  0001 C CNN
-	1    9400 2400
-	1    0    0    -1
-$EndComp
 $Comp
 L Device:D D1
@@
 	9850 3100 9850 3000
 Connection ~ 9850 3100
+$Comp
+L relay_1ct:Relay_1CT U2
+U 1 1 6062D6C5
+P 9400 2400
+F 0 "U2" H 9350 2467 50  0000 C CNN
+F 1 "Relay_1CT" H 9350 2376 50  0000 C CNN
+F 2 "OJ-SS-112LMH2_005:OJ-SS-112HM.000_1" H 9400 2400 50  0001 C CNN
+F 3 "" H 9400 2400 50  0001 C CNN
+	1    9400 2400
+	1    0    0    -1
+$EndComp
 $EndSCHEMATC
