File: ampli.kicad_pcb (KiCad board)
At the start: 2 copper layers, 110 x 100 mm, 52 parts, among them J2 Conn_01x02, J3 Conn_01x03, Q1 2N2907, Q10 TIP32, Q11 BD138, Q12 TIP31, Q13 2N2222, Q2 2N2907, Q3 2N2907, Q4 2N2222, Q5 2N2222, Q6 2N2907, Q7 2N2907, Q8 BD139, Q9 BD139, U1 Jack_Mono, U2 Relay_1CT

Commit message: test 1.1
Parts:
- moved R4 269.8 mm to (77.5, 102.9), turned to 180 degrees
- moved Q3 253.4 mm to (54.6, 110.5), turned to 180 degrees
- moved R12 229.7 mm to (92.7, 96.5), turned to 180 degrees
- moved Dz1 221.0 mm to (63.5, 102.9), turned to 180 degrees
- moved C3 197.6 mm to (144.8, 115.6)
- moved R1 197.1 mm to (71.1, 127.0), turned to 270 degrees
- moved R5 181.1 mm to (67.3, 108.0)
- moved Q13 174.2 mm to (134.6, 88.9)
- moved Q7 170.2 mm to (139.7, 108.0)
- moved C1 166.4 mm to (146.1, 124.5), turned to 270 degrees
- moved R15 166.0 mm to (99.1, 123.2)
- moved Q5 160.2 mm to (151.1, 78.7), turned to 180 degrees
- moved Q4 159.6 mm to (149.9, 88.9), turned to 270 degrees
- moved C6 151.4 mm to (146.1, 64.8)
- moved C4 150.2 mm to (125.7, 135.9)
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
Commit message: placement 1
Parts:
- moved C6 80.2 mm to (114.3, 138.4)
- moved D1 77.3 mm to (139.7, 71.1), turned to 270 degrees
- moved C2 71.9 mm to (81.3, 106.7)
- moved C1 71.2 mm to (74.9, 127.0)
- moved Q4 59.1 mm to (96.5, 114.3), turned to 90 degrees
- moved Q5 57.1 mm to (105.4, 113.0), turned to 0 degrees
- moved D2 56.3 mm to (144.8, 81.3), turned to 90 degrees
- moved R14 54.6 mm to (127.0, 90.2), turned to 270 degrees
- moved R15 54.0 mm to (147.3, 99.1), turned to 90 degrees
- moved C3 52.1 mm to (144.8, 63.5)
- moved R16 51.1 mm to (138.4, 108.0)
- moved R12 47.7 mm to (134.6, 73.7)
- moved C5 44.4 mm to (95.2, 132.1)
- moved R13 43.1 mm to (123.2, 108.0)
- moved Q8 40.9 mm to (114.3, 115.6), turned to 270 degrees
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