File: ampli.kicad_pcb (KiCad board)
At the start: 2 copper layers, 110 x 100 mm, 52 parts, among them J2 Conn_01x02, J3 Conn_01x03, Q1 2N2907, Q10 TIP32, Q11 BD138, Q12 TIP31, Q13 2N2222, Q2 2N2907, Q3 2N2907, Q4 2N2222, Q5 2N2222, Q6 2N2907, Q7 2N2907, Q8 BD139, Q9 BD139, U1 Jack_Mono, U2 Relay_1CT

Commit message: placement2
Parts:
- moved C6 89.5 mm to (95.2, 138.4)
- moved C1 77.5 mm to (68.6, 121.9), turned to 0 degrees
- moved R16 74.0 mm to (134.6, 69.8), turned to 90 degrees
- moved R6 73.4 mm to (113.0, 121.9), turned to 270 degrees
- moved C2 72.3 mm to (105.4, 130.8), turned to 90 degrees
- moved C3 62.6 mm to (138.4, 53.3)
- moved D2 62.3 mm to (139.7, 72.4), turned to 90 degrees
- moved Q5 56.4 mm to (121.9, 127.0), turned to 90 degrees
- moved Q4 55.3 mm to (120.7, 135.9)
- moved C7 46.5 mm to (86.4, 141.0)
- moved C5 43.3 mm to (95.2, 130.8)
- moved R12 39.9 mm to (72.4, 62.2), turned to 0 degrees
- moved C4 39.5 mm to (86.4, 133.3)
- moved R9 36.9 mm to (109.2, 95.2)
- moved Q7 30.7 mm to (109.2, 111.9)
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